File: PICkit.kicad_pcb (KiCad board)
At the start: 4 copper layers, 90 x 47 mm, 119 parts, among them IC1 PIC24FJ256GB106-I_PT, J1 USB_C_Receptacle_USB2.0, J2 Conn_01x06, J3 Conn_01x06, Q1 ZXTP25020CFH, Q2 2N2222A, Q3 FDC6420C, Q4 PMV48XPA2R, Q5 MMBT3904, Q6 MMBT3904, Q7 MMBT3904, Q8 MMBT3906, U1 25LC256, U2 SST25VF040B, U3 MCP1727-0802xMF, U4 SN74LVC1T45DBV, U5 74AHC1G125, U6 SN74LVC1T45DBV, U7 MCP1525-TT, U8 SN74LVC1T45DBV, U9 MCP601-xOT, Y1 12MHz

Commit message: Starting routing from scratch
Parts:
- moved R58 12.2 mm to (161.3, 102.7), turned to 0 degrees
- moved Q8 8.77 mm to (171.7, 102.3), turned to -90 degrees
- moved C17 7.58 mm to (152.5, 90.6), turned to 0 degrees
- moved Q7 5.49 mm to (164.8, 103.7), turned to 0 degrees
- moved C16 3.06 mm to (146.0, 90.6), turned to 180 degrees
- moved R57 2.87 mm to (168.3, 103.7), turned to 180 degrees
- moved U7 2.70 mm to (149.2, 89.4), turned to 90 degrees
- moved R44 1.75 mm to (187.9, 89.0)
Routing:
- net +3.3V: track 141.4 -> 17.2 mm, vias 14 -> 5
- net +5V_USB: track 112.4 -> 42.5 mm, vias 6 -> 5
- net SCLK: track 64.8 -> 0.00 mm, vias 2 -> 0
- net MISO: track 63.0 -> 0.00 mm, vias 2 -> 0
- net DATA_EN: track 62.9 -> 0.00 mm, vias 2 -> 0
- net CLK_EN: track 59.1 -> 0.00 mm, vias 2 -> 0
- net MOSI: track 58.9 -> 0.00 mm, vias 2 -> 0
- net LVP: track 0.00 -> 58.7 mm, vias 0 -> 2
- net LVP_EN: track 58.1 -> 0.00 mm, vias 3 -> 0
- net VDD_FBACK: track 55.8 -> 1.35 mm, vias 3 -> 0
- net VPP_PUMP: track 41.6 -> 0.00 mm, vias 2 -> 0
- net UTIL_SCLK: track 39.2 -> 0.00 mm, vias 3 -> 0
- net UTIL_MISO: track 38.7 -> 0.00 mm, vias 3 -> 0
- net UTIL_MOSI: track 38.2 -> 0.00 mm, vias 3 -> 0
- net VPP_TAR: track 38.5 -> 2.72 mm, vias 1 -> 0
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- added copper zone on In2.Cu, net +5V_USB

Commit message: more routing
Parts:
- moved REF** 23.6 mm to (86.2, 102.9)
- moved R5 7.84 mm to (108.8, 84.2)
- moved R6 7.54 mm to (108.8, 99.8)
- moved R16 4.92 mm to (127.6, 77.6)
- moved R17 4.92 mm to (124.6, 77.6)
- moved C15 2.30 mm to (140.7, 73.2)
- moved R25 2.30 mm to (142.2, 73.2)
- moved R26 2.30 mm to (147.9, 77.7)
- moved R27 2.30 mm to (147.9, 80.7)
- moved TH2 2.30 mm to (144.6, 73.9)
- moved Q1 2.30 mm to (141.6, 76.8)
- moved Q2 2.30 mm to (132.2, 79.7)
- moved R21 2.30 mm to (141.7, 79.7)
- moved R24 2.30 mm to (131.2, 73.8)
- moved R22 2.30 mm to (138.6, 79.7)
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Routing:
- net UTIL_SCLK: track 0.00 -> 47.5 mm, vias 0 -> 4
- net +5V_USB_GOOD: track 1.35 -> 39.4 mm, vias 0 -> 3
- net +3.3V: track 17.2 -> 49.3 mm, vias 5 -> 13
- net UTIL_MOSI: track 0.00 -> 31.7 mm, vias 0 -> 1
- net UTIL_MISO: track 0.00 -> 26.9 mm, vias 0 -> 1
- net VREF_2.5: track 1.63 -> 20.1 mm, vias 0 -> 2
- net D-: track 0.00 -> 17.1 mm, vias 0 -> 2
- net D+: track 0.00 -> 17.1 mm, vias 0 -> 2
- net UTIL_WP2: track 0.00 -> 16.4 mm
- net DBG_TX1: track 0.00 -> 12.8 mm, vias 0 -> 2
- net DBG_RX1: track 0.00 -> 12.7 mm, vias 0 -> 2
- net GND: track 24.1 -> 32.6 mm
- net Net-(J1-CC1): track 0.00 -> 7.63 mm, vias 1 -> 0
- net Net-(J1-CC2): track 0.00 -> 7.26 mm
- net ~{UTIL_CS2}: track 0.00 -> 5.14 mm
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
Commit message: Begun work on mini
Parts:
- removed C13, C14, C19, C21, C23, C24, C25, C26, C28: 0.1uF, Capacitor_SMD:C_0603_1608Metric
- removed C15: 47pF, Capacitor_SMD:C_0603_1608Metric
- removed C16, C17, C3: 1uF, Capacitor_SMD:C_0603_1608Metric
- removed C22, C27, C29: 10uF, Capacitor_Tantalum_SMD:CP_EIA-3216-18_Kemet-A
- removed C30: 47uF, Capacitor_Tantalum_SMD:CP_EIA-3216-18_Kemet-A
- removed D2: MBR0520L, Diode_SMD:D_SOD-123
- removed D3, D4, D5: 5.0V, Diode_SMD:D_0603_1608Metric
- removed D6: ZHCS1000, Package_TO_SOT_SMD:SOT-23
- removed D7: BAT54, Package_TO_SOT_SMD:SOT-23-3
- removed L1: 680uH, Inductor_SMD:L_0603_1608Metric
- removed Q1: ZXTP25020CFH, Package_TO_SOT_SMD:SOT-23-3
- removed Q2: 2N2222A, Package_TO_SOT_THT:TO-92
- removed Q3: FDC6420C, Package_TO_SOT_SMD:SuperSOT-6
- removed Q4: PMV48XPA2R, Package_TO_SOT_SMD:SOT-23-3
- removed Q5, Q6: MMBT3904, Package_TO_SOT_SMD:SOT-23
- removed Q8: MMBT3906, Package_TO_SOT_SMD:SOT-23-3
- removed R19: 330, Resistor_SMD:R_0603_1608Metric
- removed R20: 4.7k, Resistor_SMD:R_0603_1608Metric
- removed R24, R28, R29, R3, R37, R40, R45, R46, R47, R50, R52, R54, R56: 10k, Resistor_SMD:R_0603_1608Metric
- removed R25, R42, R53: 2.2k, Resistor_SMD:R_0603_1608Metric
- removed R26, R27: 2k, Resistor_SMD:R_0603_1608Metric
- removed R30, R35, R48: 100, Resistor_SMD:R_0603_1608Metric
- removed R38, R4, R44, R51: 1k, Resistor_SMD:R_0603_1608Metric
- removed R39, R49: 2.7k, Resistor_SMD:R_0603_1608Metric
- removed R41: 3.9k, Resistor_SMD:R_0603_1608Metric
- removed R55: 100k, Resistor_SMD:R_0603_1608Metric
- removed the REF** at (86.2, 102.9)
- removed TH1: MICROSMD005F, Resistor_SMD:R_0603_1608Metric
- removed TH2: Thermistor_PTC, Resistor_SMD:R_0603_1608Metric
- removed U2: SST25VF040B, Package_SO:SOIC-8_5.275x5.275mm_P1.27mm
- removed U4, U6, U8: SN74LVC1T45DBV, Package_TO_SOT_SMD:SOT-23-6
- removed U5: 74AHC1G125, Package_TO_SOT_SMD:SOT-23-5
- removed U7: MCP1525-TT, Package_TO_SOT_SMD:SOT-23
- removed U9: MCP601-xOT, Package_TO_SOT_SMD:SOT-23-5
- added R12: 3.16k, Resistor_SMD:R_0603_1608Metric, F.Cu at (170.6, 59.1)
- added R13: 100k, Resistor_SMD:R_0603_1608Metric, F.Cu at (170.6, 61.6)
- added R14: 200k, Resistor_SMD:R_0603_1608Metric, F.Cu at (170.6, 64.2)
- added R15: 10k, Resistor_SMD:R_0603_1608Metric, B.Cu at (154.8, 80.0)
- added REF**: OSHW-Logo2_7.3x6mm_SilkScreen, Symbol:OSHW-Logo2_7.3x6mm_SilkScreen, F.Cu at (147.2, 79.0)
- C10, C9: value 27pF -> 22pF
- C5, Q7, R1, R2, R43, R57, R58, R8, U1, U3: moved to B.Cu
- J2, J3: value Conn_01x06 -> Conn_01x05; footprint Connector_PinSocket_2.54mm:PinSocket_1x06_P2.54mm_Vertical -> Connector_PinSocket_2.54mm:PinSocket_1x05_P2.54mm_Vertical
- R11: value 330 -> 1k
- R18: value 100 -> 2.21k; moved to B.Cu
- R21: value 10k -> 3.92k; moved to B.Cu
- R22: value 330 -> 2.21k; moved to B.Cu
- R23: value 2.2k -> 100
- moved Y1 91.1 mm to (208.0, 81.8), turned to 90 degrees
- moved R7 86.2 mm to (170.6, 46.6)
- moved J2 76.6 mm to (179.2, 73.6)
- moved R43 71.0 mm to (175.8, 73.6), turned to 0 degrees
- moved C1 65.5 mm to (162.6, 46.6), turned to 0 degrees
- moved R11 63.4 mm to (170.6, 56.6), turned to 0 degrees
- moved C2 61.6 mm to (162.6, 49.1)
- moved R17 58.9 mm to (174.6, 46.6)
- moved C10 56.6 mm to (162.6, 69.2), turned to 0 degrees
- moved C9 55.2 mm to (162.6, 66.7), turned to 0 degrees
- moved R9 53.3 mm to (170.6, 51.6), turned to 0 degrees
- moved R8 49.9 mm to (168.3, 82.9)
- moved C11 49.1 mm to (166.6, 46.6), turned to 0 degrees
- moved R2 48.8 mm to (163.0, 75.2), turned to 0 degrees
- moved C12 48.0 mm to (166.6, 49.1), turned to 0 degrees
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Connections:
- net VPP_TAR renamed MCLR
- C9 pad 1: Net-(C9-Pad1) -> /XOSC_+
- IC1 pad 1: VPP_ON -> unconnected-(IC1-PMD5/CN63/RE5-Pad1)
- IC1 pad 11: VPP_PUMP -> unconnected-(IC1-PGEC3/AN5/C1INA/VBUSON/RP18/CN7/RB5-Pad11)
- IC1 pad 12: VDD_PUMP -> unconnected-(IC1-PGED3/AN4/C1INB/USBOEN/RP28/CN6/RB4-Pad12)
- IC1 pad 15: /RP1 -> unconnected-(IC1-PGEC1/AN1/VREF-/RP1/CN3/RB1-Pad15)
- IC1 pad 16: VREF_2.5 -> /VREF_2.5V
- IC1 pad 21: BUTTON -> unconnected-(IC1-AN8/RP8/CN26/RB8-Pad21)
- IC1 pad 22: LED_ACTIVE -> unconnected-(IC1-AN9/RP9/PMA7/CN27/RB9-Pad22)
- IC1 pad 23: LED_RESET -> unconnected-(IC1-TMS/CVREF/AN10/PMA13/CN28/RB10-Pad23)
- IC1 pad 24: LED_HALT -> unconnected-(IC1-TDO/AN11/PMA12/CN29/RB11-Pad24)
- IC1 pad 28: TMS -> unconnected-(IC1-TDI/AN13/PMA10/CTED1/CN31/RB13-Pad28)
- IC1 pad 29: DBG_TEST0 -> unconnected-(IC1-AN14/CTPLS/RP14/PMA1/CN32/RB14-Pad29)
- IC1 pad 3: +5V_USB -> unconnected-(IC1-SDA3/PMD7/CN65/RE7-Pad3)
- IC1 pad 30: REFCLKO -> unconnected-(IC1-AN15/RP29/REFO/PMA0/CN12/RB15-Pad30)
- IC1 pad 33: LVP -> unconnected-(IC1-RP16/USBID/CN71/RF3-Pad33)
- IC1 pad 4: TCK -> unconnected-(IC1-C1IND/RP21/PMA5/CN8/RG6-Pad4)
- IC1 pad 43: /RP4 -> unconnected-(IC1-DPLN/SDA1/RP4/CN54/RD9-Pad43)
- IC1 pad 44: /RP3 -> unconnected-(IC1-SCL1/RP3/PMCS2/CN55/RD10-Pad44)
- IC1 pad 49: DBG_TEST1 -> unconnected-(IC1-VCPCON/RP24/CN50/RD1-Pad49)
- IC1 pad 5: TDO -> unconnected-(IC1-C1INC/RP26/PMA4/CN9/RG7-Pad5)
- IC1 pad 54: Net-(IC1-C3INB/CN15/RD6) -> unconnected-(IC1-C3INB/CN15/RD6-Pad54)
- IC1 pad 58: UTIL_WP2 -> unconnected-(IC1-VBUSST/VCMPST1/CN68/RF0-Pad58)
- IC1 pad 59: +5V_USB_ON -> unconnected-(IC1-VCMPST2/CN69/RF1-Pad59)
- IC1 pad 6: TDI -> unconnected-(IC1-C2IND/RP19/PMA3/CN10/RG8-Pad6)
- IC1 pad 60: CLK_EN -> unconnected-(IC1-PMD0/CN58/RE0-Pad60)
- IC1 pad 61: DATA_EN -> unconnected-(IC1-PMD1/CN59/RE1-Pad61)
- IC1 pad 62: LVP_EN -> unconnected-(IC1-PMD2/CN60/RE2-Pad62)
- IC1 pad 63: SUPPLY_PWR -> Net-(IC1-PMD3/CN61/RE3)
- IC1 pad 64: +5V_USB_GOOD -> Net-(IC1-PMD4/CN62/RE4)
- IC1 pad 8: ~{UTIL_CS2} -> unconnected-(IC1-RP27/PMA2/C2INC/CN11/RG9-Pad8)
- J3 pad 2: VDD_TAR -> +3.3V
- R11 pad 1: /XOSC_+ -> +3.3V
- R11 pad 2: Net-(C9-Pad1) -> /VREF_2.5V
- R18 pad 1: LVP_VDD -> VPP_FBACK
- R18 pad 2: VDD_TAR -> GND
- R21 pad 1: VBUS -> +3.3V
- R21 pad 2: Net-(Q1-B) -> VDD_FBACK
- R22 pad 1: Net-(Q1-B) -> VDD_FBACK
- R22 pad 2: Net-(Q2-C) -> GND
- R23 pad 1: +5V_USB_ON -> VBUS_DEVICE
- R23 pad 2: Net-(Q2-B) -> VBUS
- R31 pad 2: Net-(U6-A) -> Net-(R31-Pad2)
- R32 pad 2: Net-(D4-K) -> Net-(R31-Pad2)
- R33 pad 2: Net-(U8-A) -> Net-(R33-Pad2)
- R34 pad 2: Net-(U8-A) -> Net-(R33-Pad2)
- R36 pad 2: Net-(D5-K) -> Net-(R33-Pad2)
- TH3 pad 2: Net-(D4-K) -> Net-(R31-Pad2)
- TH4 pad 2: Net-(D5-K) -> Net-(R33-Pad2)
- Y1 pad 2: Net-(C9-Pad1) -> /XOSC_+
Routing:
- net LVP: track 62.7 -> 0.00 mm, vias 2 -> 0
- net VDD_INT: track 56.4 -> 0.00 mm, vias 2 -> 0
- net +5V_USB: track 40.8 -> 0.00 mm, vias 5 -> 0
- net +5V_USB_GOOD: track 39.4 -> 0.00 mm, vias 3 -> 0
- net UTIL_SCLK: track 47.5 -> 11.1 mm, vias 4 -> 2
- net +3.3V: track 49.3 -> 15.3 mm, vias 13 -> 10
- net UTIL_MOSI: track 31.7 -> 4.60 mm
- net VDD_PUMP: track 22.6 -> 0.00 mm
- net MOSI: track 0.00 -> 21.2 mm, vias 0 -> 2
- net VBUS: track 61.1 -> 40.2 mm, vias 3 -> 2
- net VREF_2.5: track 20.1 -> 0.00 mm, vias 2 -> 0
- net MISO: track 0.00 -> 19.5 mm, vias 0 -> 2
- net SCLK: track 0.00 -> 19.1 mm, vias 0 -> 2
- net VDD_GND: track 18.6 -> 0.00 mm
- net GND: track 32.6 -> 14.9 mm
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- removed copper zone on In2.Cu, net +5V_USB
- removed copper zone on In2.Cu, net VDD_TAR
Other:
- board size 90 x 47 mm -> 50.9 x 15.4 mm
