File: PICkit.kicad_sch (KiCad schematic)
At the start: 131 parts, among them IC1 PIC24FJ256GB106-I_PT, J1 USB_C_Receptacle_USB2.0, J2 Conn_01x06, J3 Conn_01x06, Q1 ZXTP25020CFH, Q2 2N2222A, Q3 FDC6420C, Q4 PMV48XPA2R, Q5 MMBT3904, Q6 MMBT3904, Q7 MMBT3904, Q8 MMBT3906, U1 25LC256, U2 SST25VF040B, U3 MCP1727-0802xMF, U4 SN74LVC1T45DBV, U5 74AHC1G125, U6 SN74LVC1T45DBV, U7 MCP1525-TT, U8 SN74LVC1T45DBV, U9 MCP601-xOT, Y1 12MHz

Commit message: Begun work on mini
Parts:
- removed C14, C19, C21, C23, C24, C25, C26, C28: 0.1uF, Capacitor_SMD:C_0603_1608Metric, symbol Device:C_Small
- removed C15: 47pF, Capacitor_SMD:C_0603_1608Metric, symbol Device:C_Small
- removed C16, C17, C3: 1uF, Capacitor_SMD:C_0603_1608Metric, symbol Device:C_Small
- removed C22, C27, C29: 10uF, Capacitor_Tantalum_SMD:CP_EIA-3216-18_Kemet-A, symbol Device:C_Polarized_Small
- removed C30: 47uF, Capacitor_Tantalum_SMD:CP_EIA-3216-18_Kemet-A, symbol Device:C_Polarized_Small
- removed D2: MBR0520L, Diode_SMD:D_SOD-123, symbol Device:D_Small
- removed D3, D4, D5: 5.0V, Diode_SMD:D_0603_1608Metric, symbol Device:D_Schottky
- removed D6: ZHCS1000, Package_TO_SOT_SMD:SOT-23, symbol Device:D_Small
- removed D7: BAT54, Package_TO_SOT_SMD:SOT-23-3, symbol Device:D_Small
- removed J2: Conn_01x06, Connector_PinSocket_2.54mm:PinSocket_1x06_P2.54mm_Vertical, symbol Connector_Generic:Conn_01x06
- removed L1: 680uH, Inductor_SMD:L_0603_1608Metric, symbol Device:L_Small
- removed Q1: ZXTP25020CFH, Package_TO_SOT_SMD:SOT-23-3, symbol Simulation_SPICE:PNP
- removed Q2: 2N2222A, Package_TO_SOT_THT:TO-92, symbol Simulation_SPICE:NPN
- removed Q3: FDC6420C, Package_TO_SOT_SMD:SuperSOT-6, symbol Transistor_FET:FDC6330L
- removed Q4: PMV48XPA2R, Package_TO_SOT_SMD:SOT-23-3, symbol Simulation_SPICE:PMOS
- removed Q5, Q6: MMBT3904, Package_TO_SOT_SMD:SOT-23, symbol Simulation_SPICE:NPN
- removed Q8: MMBT3906, Package_TO_SOT_SMD:SOT-23-3, symbol Simulation_SPICE:PNP
- removed R24, R28, R29, R3, R37, R40, R45, R46, R47, R50, R52, R54, R56: 10k, Resistor_SMD:R_0603_1608Metric, symbol Device:R_Small
- removed R25, R42, R53: 2.2k, Resistor_SMD:R_0603_1608Metric, symbol Device:R_Small
- removed R26, R27: 2k, Resistor_SMD:R_0603_1608Metric, symbol Device:R_Small
- removed R30, R35, R48: 100, Resistor_SMD:R_0603_1608Metric, symbol Device:R_Small
- removed R38, R4, R44, R51: 1k, Resistor_SMD:R_0603_1608Metric, symbol Device:R_Small
- removed R39, R49: 2.7k, Resistor_SMD:R_0603_1608Metric, symbol Device:R_Small
- removed R41: 3.9k, Resistor_SMD:R_0603_1608Metric, symbol Device:R_Small
- removed R55: 100k, Resistor_SMD:R_0603_1608Metric, symbol Device:R_Small
- removed TH2: Thermistor_PTC, Resistor_SMD:R_0603_1608Metric, symbol Device:Thermistor_PTC
- removed TP1: ~, TestPoint:TestPoint_Plated_Hole_D2.0mm, symbol Connector:TestPoint
- removed TP10: DB0, TestPoint:TestPoint_Plated_Hole_D2.0mm, symbol Connector:TestPoint
- removed TP11: TB, TestPoint:TestPoint_Plated_Hole_D2.0mm, symbol Connector:TestPoint
- removed TP5: DB1, TestPoint:TestPoint_Plated_Hole_D2.0mm, symbol Connector:TestPoint
- removed TP6: RP1, TestPoint:TestPoint_Plated_Hole_D2.0mm, symbol Connector:TestPoint
- removed TP7: RP3, TestPoint:TestPoint_Plated_Hole_D2.0mm, symbol Connector:TestPoint
- removed TP8: RP4, TestPoint:TestPoint_Plated_Hole_D2.0mm, symbol Connector:TestPoint
- removed TP9: TMS, TestPoint:TestPoint_Plated_Hole_D2.0mm, symbol Connector:TestPoint
- removed U2: SST25VF040B, Package_SO:SOIC-8_5.275x5.275mm_P1.27mm, symbol Memory_Flash:SST25VF080B-50-4x-S2Ax
- removed U4, U6, U8: SN74LVC1T45DBV, Package_TO_SOT_SMD:SOT-23-6, symbol Logic_LevelTranslator:SN74LVC1T45DBV
- removed U5: 74AHC1G125, Package_TO_SOT_SMD:SOT-23-5, symbol 74xGxx:74AHC1G125
- removed U7: MCP1525-TT, Package_TO_SOT_SMD:SOT-23, symbol Reference_Voltage:MCP1525-TT
- removed U9: MCP601-xOT, Package_TO_SOT_SMD:SOT-23-5, symbol Amplifier_Operational:MCP601-xOT
- added J2, J3: Conn_01x05, Connector_PinSocket_2.54mm:PinSocket_1x05_P2.54mm_Vertical, symbol Connector_Generic:Conn_01x05
- added R12: 3.16k, Resistor_SMD:R_0603_1608Metric, symbol Device:R_Small
- added R13: 100k, Resistor_SMD:R_0603_1608Metric, symbol Device:R_Small
- added R14: 200k, Resistor_SMD:R_0603_1608Metric, symbol Device:R_Small
- added R15: 10k, Resistor_SMD:R_0603_1608Metric, symbol Device:R_Small
- C10, C9: value 27pF -> 22pF
- C13, R19, R20, TH1: now not fitted; now left out of the parts list
- J4: renamed from J3; now not fitted; now left out of the parts list
- R11: value 330 -> 1k
- R18: value 100 -> 2.21k
- R21: value 10k -> 3.92k
- R22: value 330 -> 2.21k
- R23: value 2.2k -> 100
Connections:
- net LVP_VDD is gone; now on net VPP_FBACK: R18.1
- net +3.3V: now also R11.1, R21.1, J2.2 (Pin_2), J3.2 (Pin_2), R13.1, R15.1
- net GND: now also R18.2, R22.2, J2.3 (Pin_3), J3.3 (Pin_3), R12.2, R14.2; no longer J4.3 (Pin_3)
- net ICSP_CLK: now also J3.5 (Pin_5); no longer J4.5 (Pin_5)
- net ICSP_DAT: now also J3.4 (Pin_4); no longer J4.4 (Pin_4)
- net ICSP_LVP: no longer J4.6 (Pin_6)
- net LVP: no longer IC1.33 (RP16/USBID/CN71/RF3)
- net MICRO_PGC: now also J2.5 (Pin_5)
- net MICRO_PGD: now also J2.4 (Pin_4)
- net MICRO_~{MCLR}: now also J2.1 (Pin_1)
- net VBUS: now also R23.2; no longer R21.1
- net VBUS_DEVICE: now also R23.1
- net VDD_FBACK: now also R21.2, R22.1
- net VPP_FBACK: now also R15.2
- net XOSC_+: now also C9.1, Y1.2; no longer R11.1
- net at R32.2, TH3.2: now also R31.2
- net at R36.2, TH4.2: now also R33.2, R34.2
- net at R20.2, TH1.2: now also R19.2
- net +5V_USB: no longer names the net of IC1.3 (SDA3/PMD7/CN65/RE7)
- net +5V_USB_GOOD: no longer names the net of IC1.64 (PMD4/CN62/RE4)
- net +5V_USB_GOOD: now also R13.2
- net +5V_USB_ON: no longer names the net of IC1.59 (VCMPST2/CN69/RF1)
- net +5V_USB_ON: no longer R23.1
- net BUTTON: no longer names the net of IC1.21 (AN8/RP8/CN26/RB8)
- net CLK_EN: no longer names the net of IC1.60 (PMD0/CN58/RE0)
- net DATA_EN: no longer names the net of IC1.61 (PMD1/CN59/RE1)
- net DBG_TEST0: no longer names the net of IC1.29 (AN14/CTPLS/RP14/PMA1/CN32/RB14)
- net DBG_TEST1: no longer names the net of IC1.49 (VCPCON/RP24/CN50/RD1)
- net LED_ACTIVE: no longer names the net of IC1.22 (AN9/RP9/PMA7/CN27/RB9)
- net LED_HALT: no longer names the net of IC1.24 (TDO/AN11/PMA12/CN29/RB11)
- net LED_RESET: no longer names the net of IC1.23 (TMS/CVREF/AN10/PMA13/CN28/RB10)
- net LVP_EN: no longer names the net of IC1.62 (PMD2/CN60/RE2)
- net REFCLKO: no longer names the net of IC1.30 (AN15/RP29/REFO/PMA0/CN12/RB15)
- net RP1: no longer names the net of IC1.15 (PGEC1/AN1/VREF-/RP1/CN3/RB1)
- net RP3: no longer names the net of IC1.44 (SCL1/RP3/PMCS2/CN55/RD10)
- net RP4: no longer names the net of IC1.43 (DPLN/SDA1/RP4/CN54/RD9)
- net SUPPLY_PWR: no longer names the net of IC1.63 (PMD3/CN61/RE3)
- net SUPPLY_PWR: now also R14.1
- net TCK: no longer names the net of IC1.4 (C1IND/RP21/PMA5/CN8/RG6)
- net TDI: no longer names the net of IC1.6 (C2IND/RP19/PMA3/CN10/RG8)
- net TDO: no longer names the net of IC1.5 (C1INC/RP26/PMA4/CN9/RG7)
- net TMS: no longer names the net of IC1.28 (TDI/AN13/PMA10/CTED1/CN31/RB13)
- net UTIL_WP2: no longer names the net of IC1.58 (VBUSST/VCMPST1/CN68/RF0)
- net VDD_PUMP: no longer names the net of IC1.12 (PGED3/AN4/C1INB/USBOEN/RP28/CN6/RB4)
- net VDD_TAR: no longer names the net of J4.2 (Pin_2)
- net VDD_TAR: no longer R18.2
- net VPP_ON: no longer names the net of IC1.1 (PMD5/CN63/RE5)
- net VPP_PUMP: no longer names the net of IC1.11 (PGEC3/AN5/C1INA/VBUSON/RP18/CN7/RB5)
- net VPP_TAR: no longer names the net of J4.1 (Pin_1)
- net VPP_TAR: no longer R57.1
- net VREF_2.5 renamed VREF_2.5V
- net VREF_2.5V: now also R11.2, R12.1
- net ~{UTIL_CS2}: no longer names the net of IC1.8 (RP27/PMA2/C2INC/CN11/RG9)
- new net MCLR: J3.1 (Pin_1), R57.1
- no-connect marks 3 -> 26
Other:
- note removed: "CODE IMAGE"
- moved on the sheet: C1, C10, C11, C12, C18, C20, C9, IC1, Q7, R16, R17, R31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
